File: ecad/motherboard/BP_4Board_Control_and_Connect.kicad_sch (KiCad schematic)
At the start: 10 parts, among them U3 TCA9544APWR, U4 CD4051BPWR4, U5 CD4051BPWR4

Commit message: Add manufacturer part numbers into Kicad Schematics
Parts:
- C3, C4, C5: MPN (none) -> C0603C104M5RACTU; Manufacturer (none) -> KEMET
- R4, R5, R6, R7: MPN (none) -> C0603FR-07100KL; Manufacturer (none) -> Yageo; notes (none) -> pull up
- U3: MPN (none) -> TCA9544APWR; Manufacturer (none) -> TI
- U4, U5: MPN (none) -> CD4051BPWR; Manufacturer (none) -> TI
Changed lines of the file:
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@@
+      (effects (font (size 1.27 1.27)) hide)
+    )
+    (property "notes" "" (at 135.89 111.76 0)
+      (effects (font (size 1.27 1.27)) hide)
+    )
+    (property "MPN" "CD4051BPWR" (at 135.89 111.76 0)
+      (effects (font (size 1.27 1.27)) hide)
+    )
+    (property "Manufacturer" "TI" (at 135.89 111.76 0)
       (effects (font (size 1.27 1.27)) hide)
     )
@@
       (effects (font (size 1.27 1.27)) hide)
     )
+    (property "notes" "" (at 104.14 49.53 0)
+      (effects (font (size 1.27 1.27)) hide)
+    )
+    (property "MPN" "C0603C104M5RACTU" (at 104.14 49.53 0)
+      (effects (font (size 1.27 1.27)) hide)
+    )
+    (property "Manufacturer" "KEMET " (at 104.14 49.53 0)
+      (effects (font (size 1.27 1.27)) hide)
+    )
     (pin "1")
     (pin "2")
@@
       (effects (font (size 1.27 1.27)) hide)
     )
+    (property "notes" "" (at 104.14 118.11 0)
+      (effects (font (size 1.27 1.27)) hide)
+    )
+    (property "MPN" "C0603C104M5RACTU" (at 104.14 118.11 0)
+      (effects (font (size 1.27 1.27)) hide)
+    )
+    (property "Manufacturer" "KEMET " (at 104.14 118.11 0)
+      (effects (font (size 1.27 1.27)) hide)
+    )
     (pin "1")
     (pin "2")
@@
     )
     (property "Datasheet" "https://www.ti.com/lit/ds/symlink/cd4051b.pdf" (at 121.92 55.88 0)
+      (effects (font (size 1.27 1.27)) hide)
+    )
+    (property "notes" "" (at 135.89 43.18 0)
+      (effects (font (size 1.27 1.27)) hide)
+    )
+    (property "MPN" "CD4051BPWR" (at 135.89 43.18 0)
+      (effects (font (size 1.27 1.27)) hide)
+    )
+    (property "Manufacturer" "TI" (at 135.89 43.18 0)
       (effects (font (size 1.27 1.27)) hide)
     )
@@
     )
     (property "Datasheet" "https://www.ti.com/lit/ds/symlink/tca9544a.pdf" (at 59.69 29.21 0)
+      (effects (font (size 1.27 1.27)) hide)
+    )
+    (property "notes" "" (at 52.07 30.48 0)
+      (effects (font (size 1.27 1.27)) hide)
+    )
+    (property "MPN" "TCA9544APWR" (at 52.07 30.48 0)
+      (effects (font (size 1.27 1.27)) hide)
+    )
+    (property "Manufacturer" "TI" (at 52.07 30.48 0)
       (effects (font (size 1.27 1.27)) hide)
     )
@@
       (effects (font (size 1.27 1.27)) hide)
     )
+    (property "notes" "pull up" (at 59.69 26.67 0)
+      (effects (font (size 1.27 1.27)) hide)
+    )
+    (property "MPN" "C0603FR-07100KL" (at 59.69 26.67 0)
+      (effects (font (size 1.27 1.27)) hide)
+    )
+    (property "Manufacturer" "Yageo" (at 59.69 26.67 0)
+      (effects (font (size 1.27 1.27)) hide)
+    )
     (pin "1")
     (pin "2")
@@
       (effects (font (size 1.27 1.27)) hide)
     )
+    (property "notes" "" (at 31.75 38.1 0)
+      (effects (font (size 1.27 1.27)) hide)
+    )
+    (property "MPN" "C0603C104M5RACTU" (at 31.75 38.1 0)
+      (effects (font (size 1.27 1.27)) hide)
+    )
+    (property "Manufacturer" "KEMET " (at 31.75 38.1 0)
+      (effects (font (size 1.27 1.27)) hide)
+    )
     (pin "1")
     (pin "2")
@@
       (effects (font (size 1.27 1.27)) hide)
     )
+    (property "notes" "pull up" (at 82.55 26.67 0)
+      (effects (font (size 1.27 1.27)) hide)
+    )
+    (property "MPN" "C0603FR-07100KL" (at 82.55 26.67 0)
+      (effects (font (size 1.27 1.27)) hide)
+    )
+    (property "Manufacturer" "Yageo" (at 82.55 26.67 0)
+      (effects (font (size 1.27 1.27)) hide)
+    )
     (pin "1")
     (pin "2")
@@
       (effects (font (size 1.27 1.27)) hide)
     )
+    (property "notes" "pull up" (at 67.31 26.67 0)
+      (effects (font (size 1.27 1.27)) hide)
+    )
+    (property "MPN" "C0603FR-07100KL" (at 67.31 26.67 0)
+      (effects (font (size 1.27 1.27)) hide)
+    )
+    (property "Manufacturer" "Yageo" (at 67.31 26.67 0)
+      (effects (font (size 1.27 1.27)) hide)
+    )
     (pin "1")
     (pin "2")
@@
       (effects (font (size 1.27 1.27)) hide)
     )
+    (property "notes" "pull up" (at 74.93 26.67 0)
+      (effects (font (size 1.27 1.27)) hide)
+    )
+    (property "MPN" "C0603FR-07100KL" (at 74.93 26.67 0)
+      (effects (font (size 1.27 1.27)) hide)
+    )
+    (property "Manufacturer" "Yageo" (at 74.93 26.67 0)
+      (effects (font (size 1.27 1.27)) hide)
+    )
