File: ecad/motherboard/BP_Channel.kicad_sch (KiCad schematic)
At the start: 18 parts, among them J6 Amphenol_10061913-xx0, U21 NE5532, U22 TLP4026G, U23 TLP4026G

Commit message: Add manufacturer part numbers into Kicad Schematics
Parts:
- C25, C26: MPN (none) -> GRM55DR72E105KW01L; Manufacturer (none) -> Murata
- C27, C28: MPN (none) -> C0603C104M5RACTU; Manufacturer (none) -> KEMET
- J6: MPN (none) -> 10061913-110PLF; Manufacturer (none) -> Amphenol
- R52, R53, R58, R59: MPN (none) -> RT0603FRE0722KL; Manufacturer (none) -> Yageo; notes (none) -> Thin Film
- R54, R55, R56, R57: MPN (none) -> RC0603FR-073K3L; Manufacturer (none) -> Yageo
- R60, R61: MPN (none) -> RT0603FRE071KL; Manufacturer (none) -> Yageo; notes (none) -> Thin Film
- U21: MPN (none) -> NE5532ADR; Manufacturer (none) -> TI
- U22, U23: MPN (none) -> CPC2317NTR; Manufacturer (none) -> IXYS
Changed lines of the file:
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@@
+      (effects (font (size 1.27 1.27)) hide)
+    )
+    (property "notes" "" (at 180.34 40.64 0)
+      (effects (font (size 1.27 1.27)) hide)
+    )
+    (property "MPN" "NE5532ADR" (at 180.34 40.64 0)
+      (effects (font (size 1.27 1.27)) hide)
+    )
+    (property "Manufacturer" "TI" (at 180.34 40.64 0)
       (effects (font (size 1.27 1.27)) hide)
     )
@@
       (effects (font (size 1.27 1.27)) hide)
     )
+    (property "notes" "" (at 180.34 135.89 0)
+      (effects (font (size 1.27 1.27)) hide)
+    )
+    (property "MPN" "NE5532ADR" (at 180.34 135.89 0)
+      (effects (font (size 1.27 1.27)) hide)
+    )
+    (property "Manufacturer" "TI" (at 180.34 135.89 0)
+      (effects (font (size 1.27 1.27)) hide)
+    )
     (pin "1")
     (pin "2")
@@
       (effects (font (size 1.27 1.27)) hide)
     )
+    (property "notes" "Thin Film" (at 165.1 38.1 0)
+      (effects (font (size 1.27 1.27)) hide)
+    )
+    (property "MPN" "RT0603FRE0722KL" (at 165.1 38.1 0)
+      (effects (font (size 1.27 1.27)) hide)
+    )
+    (property "Manufacturer" "Yageo" (at 165.1 38.1 0)
+      (effects (font (size 1.27 1.27)) hide)
+    )
     (pin "1")
     (pin "2")
@@
       (effects (font (size 1.27 1.27)) hide)
     )
+    (property "notes" "" (at 158.75 38.1 0)
+      (effects (font (size 1.27 1.27)) hide)
+    )
+    (property "MPN" "GRM55DR72E105KW01L" (at 158.75 38.1 0)
+      (effects (font (size 1.27 1.27)) hide)
+    )
+    (property "Manufacturer" "Murata" (at 158.75 38.1 0)
+      (effects (font (size 1.27 1.27)) hide)
+    )
     (pin "1")
     (pin "2")
@@
       (effects (font (size 1.27 1.27)) hide)
     )
+    (property "notes" "Thin Film" (at 198.12 33.02 0)
+      (effects (font (size 1.27 1.27)) hide)
+    )
+    (property "MPN" "RT0603FRE0722KL" (at 198.12 33.02 0)
+      (effects (font (size 1.27 1.27)) hide)
+    )
+    (property "Manufacturer" "Yageo" (at 198.12 33.02 0)
+      (effects (font (size 1.27 1.27)) hide)
+    )
     (pin "1")
     (pin "2")
@@
     )
     (property "Datasheet" "~" (at 208.28 40.64 0)
+      (effects (font (size 1.27 1.27)) hide)
+    )
+    (property "notes" "Thin Film" (at 208.28 40.64 0)
+      (effects (font (size 1.27 1.27)) hide)
+    )
+    (property "MPN" "RT0603FRE071KL" (at 208.28 40.64 0)
+      (effects (font (size 1.27 1.27)) hide)
+    )
+    (property "Manufacturer" "Yageo" (at 208.28 40.64 0)
       (effects (font (size 1.27 1.27)) hide)
     )
@@
       (effects (font (size 1.27 1.27)) hide)
     )
+    (property "notes" "" (at 171.45 137.16 0)
+      (effects (font (size 1.27 1.27)) hide)
+    )
+    (property "MPN" "C0603C104M5RACTU" (at 171.45 137.16 0)
+      (effects (font (size 1.27 1.27)) hide)
+    )
+    (property "Manufacturer" "KEMET " (at 171.45 137.16 0)
+      (effects (font (size 1.27 1.27)) hide)
+    )
     (pin "1")
     (pin "2")
@@
       (effects (font (size 1.27 1.27)) hide)
     )
+    (property "notes" "" (at 189.23 137.16 0)
+      (effects (font (size 1.27 1.27)) hide)
+    )
+    (property "MPN" "C0603C104M5RACTU" (at 189.23 137.16 0)
+      (effects (font (size 1.27 1.27)) hide)
+    )
+    (property "Manufacturer" "KEMET " (at 189.23 137.16 0)
+      (effects (font (size 1.27 1.27)) hide)
+    )
     (pin "1")
     (pin "2")
@@
       (effects (font (size 1.27 1.27)) hide)
     )
+    (property "notes" "" (at 184.15 60.96 0)
+      (effects (font (size 1.27 1.27)) hide)
+    )
+    (property "MPN" "RC0603FR-073K3L" (at 184.15 60.96 0)
+      (effects (font (size 1.27 1.27)) hide)
+    )
+    (property "Manufacturer" "Yageo" (at 184.15 60.96 0)
+      (effects (font (size 1.27 1.27)) hide)
+    )
     (pin "1")
     (pin "2")
@@
       (effects (font (size 1.27 1.27)) hide)
     )
+    (property "notes" "" (at 189.23 68.58 0)
+      (effects (font (size 1.27 1.27)) hide)
+    )
+    (property "MPN" "RC0603FR-073K3L" (at 189.23 68.58 0)
+      (effects (font (size 1.27 1.27)) hide)
+    )
+    (property "Manufacturer" "Yageo" (at 189.23 68.58 0)
+      (effects (font (size 1.27 1.27)) hide)
+    )
     (pin "1")
     (pin "2")
@@
     )
     (property "Datasheet" "http://www.ti.com/lit/ds/symlink/ne5532.pdf" (at 204.47 87.63 0)
+      (effects (font (size 1.27 1.27)) hide)
+    )
+    (property "notes" "" (at 180.34 91.44 0)
+      (effects (font (size 1.27 1.27)) hide)
+    )
+    (property "MPN" "NE5532ADR" (at 180.34 91.44 0)
+      (effects (font (size 1.27 1.27)) hide)
+    )
+    (property "Manufacturer" "TI" (at 180.34 91.44 0)
       (effects (font (size 1.27 1.27)) hide)
     )
@@
       (effects (font (size 1.27 1.27)) hide)
     )
+    (property "notes" "Thin Film" (at 165.1 88.9 0)
+      (effects (font (size 1.27 1.27)) hide)
+    )
+    (property "MPN" "RT0603FRE0722KL" (at 165.1 88.9 0)
+      (effects (font (size 1.27 1.27)) hide)
+    )
+    (property "Manufacturer" "Yageo" (at 165.1 88.9 0)
+      (effects (font (size 1.27 1.27)) hide)
+    )
     (pin "1")
     (pin "2")
@@
       (effects (font (size 1.27 1.27)) hide)
     )
+    (property "notes" "" (at 158.75 88.9 0)
+      (effects (font (size 1.27 1.27)) hide)
+    )
+    (property "MPN" "GRM55DR72E105KW01L" (at 158.75 88.9 0)
+      (effects (font (size 1.27 1.27)) hide)
+    )
+    (property "Manufacturer" "Murata" (at 158.75 88.9 0)
+      (effects (font (size 1.27 1.27)) hide)
+    )
     (pin "1")
     (pin "2")
@@
       (effects (font (size 1.27 1.27)) hide)
     )
+    (property "notes" "Thin Film" (at 198.12 83.82 0)
+      (effects (font (size 1.27 1.27)) hide)
+    )
+    (property "MPN" "RT0603FRE0722KL" (at 198.12 83.82 0)
+      (effects (font (size 1.27 1.27)) hide)
+    )
+    (property "Manufacturer" "Yageo" (at 198.12 83.82 0)
+      (effects (font (size 1.27 1.27)) hide)
+    )
     (pin "1")
     (pin "2")
@@
     )
     (property "Datasheet" "~" (at 208.28 91.44 0)
+      (effects (font (size 1.27 1.27)) hide)
+    )
+    (property "notes" "Thin Film" (at 208.28 91.44 0)
+      (effects (font (size 1.27 1.27)) hide)
+    )
+    (property "MPN" "RT0603FRE071KL" (at 208.28 91.44 0)
+      (effects (font (size 1.27 1.27)) hide)
+    )
+    (property "Manufacturer" "Yageo" (at 208.28 91.44 0)
       (effects (font (size 1.27 1.27)) hide)
     )
@@
       (effects (font (size 1.27 1.27)) hide)
     )
+    (property "notes" "" (at 184.15 111.76 0)
+      (effects (font (size 1.27 1.27)) hide)
+    )
+    (property "MPN" "RC0603FR-073K3L" (at 184.15 111.76 0)
+      (effects (font (size 1.27 1.27)) hide)
+    )
+    (property "Manufacturer" "Yageo" (at 184.15 111.76 0)
+      (effects (font (size 1.27 1.27)) hide)
+    )
     (pin "1")
     (pin "2")
@@
     )
     (property "Datasheet" "~" (at 189.23 119.38 0)
+      (effects (font (size 1.27 1.27)) hide)
+    )
+    (property "notes" "" (at 189.23 119.38 0)
+      (effects (font (size 1.27 1.27)) hide)
+    )
+    (property "MPN" "RC0603FR-073K3L" (at 189.23 119.38 0)
+      (effects (font (size 1.27 1.27)) hide)
+    )
+    (property "Manufacturer" "Yageo" (at 189.23 119.38 0)
       (effects (font (size 1.27 1.27)) hide)
     )
@@
     )
     (property "Datasheet" "" (at 204.47 44.45 0)
+      (effects (font (size 1.27 1.27)) hide)
+    )
+    (property "notes" "" (at 196.85 52.07 0)
+      (effects (font (size 1.27 1.27)) hide)
+    )
+    (property "MPN" "CPC2317NTR" (at 196.85 52.07 0)
+      (effects (font (size 1.27 1.27)) hide)
+    )
+    (property "Manufacturer" "IXYS" (at 196.85 52.07 0)
       (effects (font (size 1.27 1.27)) hide)
     )
@@
     )
     (property "Datasheet" "" (at 92.71 82.55 0)
+      (effects (font (size 1.27 1.27)) hide)
+    )
+    (property "notes" "" (at 92.71 82.55 0)
+      (effects (font (size 1.27 1.27)) hide)
+    )
+    (property "MPN" "10061913-110PLF" (at 92.71 82.55 0)
+      (effects (font (size 1.27 1.27)) hide)
+    )
+    (property "Manufacturer" "Amphenol" (at 92.71 82.55 0)
       (effects (font (size 1.27 1.27)) hide)
     )
@@
       (effects (font (size 1.27 1.27)) hide)
     )
+    (property "notes" "" (at 196.85 102.87 0)
+      (effects (font (size 1.27 1.27)) hide)
+    )
+    (property "MPN" "CPC2317NTR" (at 196.85 102.87 0)
+      (effects (font (size 1.27 1.27)) hide)
+    )
+    (property "Manufacturer" "IXYS" (at 196.85 102.87 0)
+      (effects (font (size 1.27 1.27)) hide)
+    )
