File: ecad/motherboard/motherboard.kicad_pcb (KiCad board)
At the start: 2 copper layers, 199.5 x 99.5 mm, 207 parts, among them J1 B6B-XH-A(LF)(SN), J2 Amphenol_10061913-xx0, J3 Amphenol_10061913-xx0, J4 Amphenol_10061913-xx0, J5 Amphenol_10061913-xx0, J6 Amphenol_10061913-xx0, J7 Amphenol_10061913-xx0, J8 Amphenol_10061913-xx0, J9 Amphenol_10061913-xx0, U1 CD4051BPWR4, U10 TLP4026G, U11 TLP4026G, U12 NE5532, U13 TLP4026G, U14 TLP4026G, U15 NE5532, U16 TLP4026G, U17 TLP4026G, U18 TCA9544APWR, U19 CD4051BPWR4, U2 NodeMCU ESP-32S, U20 CD4051BPWR4, U21 NE5532, U22 TLP4026G, U23 TLP4026G, U24 NE5532, U25 TLP4026G, U26 TLP4026G, U27 NE5532, U28 TLP4026G, U29 TLP4026G, U3 TCA9544APWR, U30 NE5532, U31 TLP4026G, U32 TLP4026G, U33 NE5532, U34 PGA231x, U4 CD4051BPWR4, U5 CD4051BPWR4, U6 NE5532, U7 TLP4026G, U8 TLP4026G, U9 NE5532

Commit message: Fix missing mask and paste layers on support pad of PCI connector. Open mask expansion slightly and close paste slightly.
Other:
- rule pad_to_mask_clearance: 0 -> 0.03
Changed lines of the file:
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@@
       (dielectric_constraints no)
     )
-    (pad_to_mask_clearance 0)
+    (pad_to_mask_clearance 0.03)
+    (pad_to_paste_clearance -0.1)
     (grid_origin 58 150.25)
     (pcbplotparams
@@
       )
       (stroke (width 0.1) (type solid)) (fill solid) (layer "F.Cu"))
+    (fp_poly
+      (pts
+        (xy 11.8 2.45)
+        (xy 11.8 -2.4)
+        (xy 8.9 -2.4)
+        (xy 8.9 -1)
+        (xy 9.6 -1)
+        (xy 10.15 -0.425)
+        (xy 10.15 0.425)
+        (xy 9.6 1)
+        (xy 8.9 1)
+        (xy 8.9 2.45)
+      )
+      (stroke (width 0.1) (type solid)) (fill solid) (layer "F.Paste"))
     (fp_line (start -12.45 -5.1) (end 8.15 -5.1)
       (stroke (width 0.12) (type solid)) (layer "F.SilkS"))
@@
     (fp_poly
       (pts
+        (xy 11.8 2.45)
+        (xy 11.8 -2.4)
+        (xy 8.9 -2.4)
+        (xy 8.9 -1)
+        (xy 8.9 1)
+        (xy 8.9 2.45)
+      )
+      (stroke (width 0.1) (type solid)) (fill solid) (layer "F.Mask"))
+    (fp_poly
+      (pts
         (xy -16.256 -2.54)
         (xy -12.192 -2.54)
@@
       )
       (stroke (width 0.1) (type solid)) (fill solid) (layer "F.Cu"))
+    (fp_poly
+      (pts
+        (xy 11.8 2.45)
+        (xy 11.8 -2.4)
+        (xy 8.9 -2.4)
+        (xy 8.9 -1)
+        (xy 9.6 -1)
+        (xy 10.15 -0.425)
+        (xy 10.15 0.425)
+        (xy 9.6 1)
+        (xy 8.9 1)
+        (xy 8.9 2.45)
+      )
+      (stroke (width 0.1) (type solid)) (fill solid) (layer "F.Paste"))
     (fp_line (start -12.45 -5.1) (end 8.15 -5.1)
       (stroke (width 0.12) (type solid)) (layer "F.SilkS"))
@@
     (fp_poly
       (pts
+        (xy 11.8 2.45)
+        (xy 11.8 -2.4)
+        (xy 8.9 -2.4)
+        (xy 8.9 -1)
+        (xy 8.9 1)
+        (xy 8.9 2.45)
+      )
+      (stroke (width 0.1) (type solid)) (fill solid) (layer "F.Mask"))
+    (fp_poly
+      (pts
         (xy -16.256 -2.54)
         (xy -12.192 -2.54)
@@
       )
       (stroke (width 0.1) (type solid)) (fill solid) (layer "F.Cu"))
+    (fp_poly
+      (pts
+        (xy 11.8 2.45)
+        (xy 11.8 -2.4)
+        (xy 8.9 -2.4)
+        (xy 8.9 -1)
+        (xy 9.6 -1)
+        (xy 10.15 -0.425)
+        (xy 10.15 0.425)
+        (xy 9.6 1)
+        (xy 8.9 1)
+        (xy 8.9 2.45)
+      )
+      (stroke (width 0.1) (type solid)) (fill solid) (layer "F.Paste"))
     (fp_line (start -12.45 -5.1) (end 8.15 -5.1)
       (stroke (width 0.12) (type solid)) (layer "F.SilkS"))
@@
     (fp_poly
       (pts
+        (xy 11.8 2.45)
+        (xy 11.8 -2.4)
+        (xy 8.9 -2.4)
+        (xy 8.9 -1)
+        (xy 8.9 1)
+        (xy 8.9 2.45)
+      )
+      (stroke (width 0.1) (type solid)) (fill solid) (layer "F.Mask"))
+    (fp_poly
+      (pts
         (xy -16.256 -2.54)
         (xy -12.192 -2.54)
@@
       )
       (stroke (width 0.1) (type solid)) (fill solid) (layer "F.Cu"))
+    (fp_poly
+      (pts
+        (xy 11.8 2.45)
+        (xy 11.8 -2.4)
+        (xy 8.9 -2.4)
+        (xy 8.9 -1)
+        (xy 9.6 -1)
+        (xy 10.15 -0.425)
+        (xy 10.15 0.425)
+        (xy 9.6 1)
+        (xy 8.9 1)
+        (xy 8.9 2.45)
+      )
+      (stroke (width 0.1) (type solid)) (fill solid) (layer "F.Paste"))
     (fp_line (start -12.45 -5.1) (end 8.15 -5.1)
       (stroke (width 0.12) (type solid)) (layer "F.SilkS"))
@@
     (fp_poly
       (pts
+        (xy 11.8 2.45)
+        (xy 11.8 -2.4)
+        (xy 8.9 -2.4)
+        (xy 8.9 -1)
+        (xy 8.9 1)
+        (xy 8.9 2.45)
+      )
+      (stroke (width 0.1) (type solid)) (fill solid) (layer "F.Mask"))
+    (fp_poly
+      (pts
         (xy -16.256 -2.54)
         (xy -12.192 -2.54)
@@
       )
       (stroke (width 0.1) (type solid)) (fill solid) (layer "F.Cu"))
+    (fp_poly
+      (pts
+        (xy 11.8 2.45)
+        (xy 11.8 -2.4)
+        (xy 8.9 -2.4)
+        (xy 8.9 -1)
+        (xy 9.6 -1)
+        (xy 10.15 -0.425)
+        (xy 10.15 0.425)
+        (xy 9.6 1)
+        (xy 8.9 1)
+        (xy 8.9 2.45)
+      )
+      (stroke (width 0.1) (type solid)) (fill solid) (layer "F.Paste"))
     (fp_line (start -12.45 -5.1) (end 8.15 -5.1)
       (stroke (width 0.12) (type solid)) (layer "F.SilkS"))
@@
     (fp_poly
       (pts
+        (xy 11.8 2.45)
+        (xy 11.8 -2.4)
+        (xy 8.9 -2.4)
+        (xy 8.9 -1)
+        (xy 8.9 1)
+        (xy 8.9 2.45)
+      )
+      (stroke (width 0.1) (type solid)) (fill solid) (layer "F.Mask"))
+    (fp_poly
+      (pts
         (xy -16.256 -2.54)
         (xy -12.192 -2.54)
@@
       )
       (stroke (width 0.1) (type solid)) (fill solid) (layer "F.Cu"))
+    (fp_poly
+      (pts
+        (xy 11.8 2.45)
+        (xy 11.8 -2.4)
+        (xy 8.9 -2.4)
+        (xy 8.9 -1)
+        (xy 9.6 -1)
+        (xy 10.15 -0.425)
+        (xy 10.15 0.425)
+        (xy 9.6 1)
+        (xy 8.9 1)
+        (xy 8.9 2.45)
+      )
+      (stroke (width 0.1) (type solid)) (fill solid) (layer "F.Paste"))
     (fp_line (start -12.45 -5.1) (end 8.15 -5.1)
       (stroke (width 0.12) (type solid)) (layer "F.SilkS"))
@@
     (fp_poly
       (pts
+        (xy 11.8 2.45)
+        (xy 11.8 -2.4)
+        (xy 8.9 -2.4)
+        (xy 8.9 -1)
+        (xy 8.9 1)
+        (xy 8.9 2.45)
+      )
+      (stroke (width 0.1) (type solid)) (fill solid) (layer "F.Mask"))
+    (fp_poly
+      (pts
         (xy -16.256 -2.54)
         (xy -12.192 -2.54)
@@
       )
       (stroke (width 0.1) (type solid)) (fill solid) (layer "F.Cu"))
+    (fp_poly
+      (pts
+        (xy 11.8 2.45)
+        (xy 11.8 -2.4)
+        (xy 8.9 -2.4)
+        (xy 8.9 -1)
+        (xy 9.6 -1)
+        (xy 10.15 -0.425)
+        (xy 10.15 0.425)
+        (xy 9.6 1)
+        (xy 8.9 1)
+        (xy 8.9 2.45)
+      )
+      (stroke (width 0.1) (type solid)) (fill solid) (layer "F.Paste"))
     (fp_line (start -12.45 -5.1) (end 8.15 -5.1)
       (stroke (width 0.12) (type solid)) (layer "F.SilkS"))
@@
     (fp_poly
       (pts
+        (xy 11.8 2.45)
+        (xy 11.8 -2.4)
+        (xy 8.9 -2.4)
+        (xy 8.9 -1)
+        (xy 8.9 1)
+        (xy 8.9 2.45)
+      )
+      (stroke (width 0.1) (type solid)) (fill solid) (layer "F.Mask"))
+    (fp_poly
+      (pts
         (xy -16.256 -2.54)
         (xy -12.192 -2.54)
@@
       )
       (stroke (width 0.1) (type solid)) (fill solid) (layer "F.Cu"))
+    (fp_poly
+      (pts
+        (xy 11.8 2.45)
+        (xy 11.8 -2.4)
+        (xy 8.9 -2.4)
+        (xy 8.9 -1)
+        (xy 9.6 -1)
+        (xy 10.15 -0.425)
+        (xy 10.15 0.425)
+        (xy 9.6 1)
+        (xy 8.9 1)
+        (xy 8.9 2.45)
+      )
+      (stroke (width 0.1) (type solid)) (fill solid) (layer "F.Paste"))
     (fp_line (start -12.45 -5.1) (end 8.15 -5.1)
       (stroke (width 0.12) (type solid)) (layer "F.SilkS"))
@@
     (fp_poly
       (pts
+        (xy 11.8 2.45)
+        (xy 11.8 -2.4)
+        (xy 8.9 -2.4)
+        (xy 8.9 -1)
+        (xy 8.9 1)
+        (xy 8.9 2.45)
+      )
+      (stroke (width 0.1) (type solid)) (fill solid) (layer "F.Mask"))
+    (fp_poly
+      (pts
